File: hardware_mx/beat_sequencer.kicad_pcb (KiCad board)
At the start: 2 copper layers, 304.2 x 124.6 mm, 338 parts, among them Q1 2N7002, SW1 SW_SPST, SW10 SW_SPST, SW11 SW_SPST, SW12 SW_SPST, SW13 SW_SPST, SW14 SW_SPST, SW15 SW_SPST, SW16 SW_SPST, SW17 SW_SPST, SW18 SW_SPST, SW19 SW_SPST, SW2 SW_SPST, SW20 SW_SPST, SW21 SW_SPST, SW22 SW_SPST, SW23 SW_SPST, SW24 SW_SPST, SW25 SW_SPST, SW26 SW_SPST, SW27 SW_SPST, SW28 SW_SPST, SW29 SW_SPST, SW3 SW_SPST, SW30 SW_SPST, SW31 SW_SPST, SW32 SW_SPST, SW33 SW_SPST, SW34 SW_SPST, SW35 SW_SPST, SW36 SW_SPST, SW37 SW_SPST, SW38 SW_SPST, SW39 SW_SPST, SW4 SW_SPST, SW40 SW_SPST, SW41 SW_SPST, SW42 SW_SPST, SW43 SW_SPST, SW44 SW_SPST, SW45 SW_SPST, SW46 SW_SPST, SW47 SW_SPST, SW48 SW_SPST, SW49 SW_SPST, SW5 SW_SPST, SW50 SW_SPST, SW51 SW_SPST, SW52 SW_SPST, SW53 SW_SPST, SW54 SW_SPST, SW55 SW_SPST, SW56 SW_SPST, SW57 SW_SPST, SW58 SW_SPST, SW59 SW_SPST, SW6 SW_SPST, SW60 SW_SPST, SW61 SW_SPST, SW62 SW_SPST, SW63 SW_SPST, SW64 SW_SPST, SW65 SW_SPST, SW66 SW_SPST, SW67 SW_SPST, SW68 SW_SPST, SW69 SW_SPST, SW7 SW_SPST, SW70 SW_SPST, SW71 SW_SPST, SW72 SW_SPST, SW73 SW_SPST, SW74 RotaryEncoder_Switch_MP, SW75 SW_SPST, SW76 SW_SPST, SW77 SW_SPST, SW78 SW_SPST, SW79 SW_SPST, SW8 SW_SPST, SW80 SW_SPST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

Commit message: Add mosfets to columns
Parts:
- added Q2: 2N7002, Package_TO_SOT_SMD:SOT-23, B.Cu at (234.0, 117.8)
- added Q3: 2N7002, Package_TO_SOT_SMD:SOT-23, B.Cu at (238.2, 120.1)
- added Q4: 2N7002, Package_TO_SOT_SMD:SOT-23, B.Cu at (242.6, 122.3)
- added Q5: 2N7002, Package_TO_SOT_SMD:SOT-23, B.Cu at (251.3, 121.4)
- added Q6: 2N7002, Package_TO_SOT_SMD:SOT-23, B.Cu at (256.7, 122.2)
- added Q7: 2N7002, Package_TO_SOT_SMD:SOT-23, B.Cu at (276.3, 121.6)
- added Q8: 2N7002, Package_TO_SOT_SMD:SOT-23, B.Cu at (281.8, 121.6)
- added Q9: 2N7002, Package_TO_SOT_SMD:SOT-23, B.Cu at (287.2, 121.6)
- A1: value RaspberryPi_Pico -> RaspberryPi_Pico2
Connections:
- SW10 pad 2: C1 -> Net-(Q2-D)
- SW11 pad 2: C1 -> Net-(Q2-D)
- SW12 pad 2: C2 -> Net-(Q3-D)
- SW13 pad 2: C2 -> Net-(Q3-D)
- SW14 pad 2: C3 -> Net-(Q4-D)
- SW15 pad 2: C3 -> Net-(Q4-D)
- SW16 pad 2: C4 -> Net-(Q5-D)
- SW17 pad 2: C4 -> Net-(Q5-D)
- SW18 pad 2: C5 -> Net-(Q6-D)
- SW19 pad 2: C5 -> Net-(Q6-D)
- SW2 pad 2: C2 -> Net-(Q3-D)
- SW20 pad 2: C5 -> Net-(Q6-D)
- SW21 pad 2: C5 -> Net-(Q6-D)
- SW22 pad 2: C6 -> Net-(Q7-D)
- SW23 pad 2: C6 -> Net-(Q7-D)
- SW24 pad 2: C6 -> Net-(Q7-D)
- SW25 pad 2: C6 -> Net-(Q7-D)
- SW26 pad 2: C7 -> Net-(Q8-D)
- SW27 pad 2: C7 -> Net-(Q8-D)
- SW28 pad 2: C7 -> Net-(Q8-D)
- SW29 pad 2: C7 -> Net-(Q8-D)
- SW3 pad 2: C1 -> Net-(Q2-D)
- SW30 pad 2: C8 -> Net-(Q9-D)
- SW31 pad 2: C8 -> Net-(Q9-D)
- SW32 pad 2: C8 -> Net-(Q9-D)
- SW33 pad 2: C8 -> Net-(Q9-D)
- SW34 pad 2: C1 -> Net-(Q2-D)
- SW35 pad 2: C1 -> Net-(Q2-D)
- SW36 pad 2: C1 -> Net-(Q2-D)
- SW37 pad 2: C1 -> Net-(Q2-D)
- SW38 pad 2: C2 -> Net-(Q3-D)
- SW39 pad 2: C2 -> Net-(Q3-D)
- SW4 pad 2: C3 -> Net-(Q4-D)
- SW40 pad 2: C2 -> Net-(Q3-D)
- SW41 pad 2: C2 -> Net-(Q3-D)
- SW42 pad 2: C3 -> Net-(Q4-D)
- SW43 pad 2: C3 -> Net-(Q4-D)
- SW44 pad 2: C3 -> Net-(Q4-D)
- SW45 pad 2: C3 -> Net-(Q4-D)
- SW46 pad 2: C4 -> Net-(Q5-D)
- SW47 pad 2: C4 -> Net-(Q5-D)
- SW48 pad 2: C4 -> Net-(Q5-D)
- SW49 pad 2: C4 -> Net-(Q5-D)
- SW5 pad 2: C4 -> Net-(Q5-D)
- SW50 pad 2: C5 -> Net-(Q6-D)
- SW51 pad 2: C5 -> Net-(Q6-D)
- SW52 pad 2: C5 -> Net-(Q6-D)
- SW53 pad 2: C5 -> Net-(Q6-D)
- SW54 pad 2: C6 -> Net-(Q7-D)
- SW55 pad 2: C6 -> Net-(Q7-D)
- SW56 pad 2: C6 -> Net-(Q7-D)
- SW57 pad 2: C6 -> Net-(Q7-D)
- SW58 pad 2: C7 -> Net-(Q8-D)
- SW59 pad 2: C7 -> Net-(Q8-D)
- SW6 pad 2: C1 -> Net-(Q2-D)
- SW60 pad 2: C7 -> Net-(Q8-D)
- SW61 pad 2: C7 -> Net-(Q8-D)
- SW62 pad 2: C8 -> Net-(Q9-D)
- SW63 pad 2: C8 -> Net-(Q9-D)
- SW64 pad 2: C8 -> Net-(Q9-D)
- SW65 pad 2: C8 -> Net-(Q9-D)
- SW66 pad 2: C1 -> Net-(Q2-D)
- SW67 pad 2: C2 -> Net-(Q3-D)
- SW68 pad 2: C3 -> Net-(Q4-D)
- SW69 pad 2: C4 -> Net-(Q5-D)
- SW7 pad 2: C2 -> Net-(Q3-D)
- SW70 pad 2: C5 -> Net-(Q6-D)
- SW71 pad 2: C6 -> Net-(Q7-D)
- SW72 pad 2: C7 -> Net-(Q8-D)
- SW73 pad 2: C8 -> Net-(Q9-D)
- SW75 pad 2: C1 -> Net-(Q2-D)
- SW76 pad 2: C2 -> Net-(Q3-D)
- SW77 pad 2: C3 -> Net-(Q4-D)
- SW78 pad 2: C4 -> Net-(Q5-D)
- SW79 pad 2: C5 -> Net-(Q6-D)
- SW8 pad 2: C3 -> Net-(Q4-D)
- SW80 pad 2: C6 -> Net-(Q7-D)
- SW81 pad 2: C7 -> Net-(Q8-D)
- SW82 pad 2: C8 -> Net-(Q9-D)
- SW9 pad 2: C4 -> Net-(Q5-D)
Routing:
- net C1: track 479.0 -> 111.8 mm, vias 5 -> 3
- net Net-(Q2-D): track 0.00 -> 366.2 mm, vias 0 -> 4
- net Net-(Q3-D): track 0.00 -> 348.9 mm, vias 0 -> 4
- net C2: track 460.8 -> 118.8 mm, vias 5 -> 3
- net C5: track 436.5 -> 102.3 mm, vias 6 -> 3
- net Net-(Q5-D): track 0.00 -> 332.9 mm, vias 0 -> 5
- net Net-(Q8-D): track 0.00 -> 332.8 mm, vias 0 -> 5
- net Net-(Q9-D): track 0.00 -> 332.4 mm, vias 0 -> 5
- net Net-(Q4-D): track 0.00 -> 332.3 mm, vias 0 -> 4
- net Net-(Q7-D): track 0.00 -> 332.3 mm, vias 0 -> 5
- net Net-(Q6-D): track 0.00 -> 332.0 mm, vias 0 -> 5
- net C4: track 436.6 -> 109.4 mm, vias 6 -> 3
- net C3: track 445.4 -> 126.4 mm, vias 6 -> 3
- net C7: track 334.4 -> 39.6 mm, vias 4 -> 3
- net C8: track 334.4 -> 40.6 mm, vias 4 -> 3
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